File: Timeline/Timeline.kicad_sch (KiCad schematic)
At the start: 118 parts, among them M1 Vibration, SW1 RotaryEncoder_Switch, SW100 SW_Push, SW101 SW_Push, SW102 SW_Push, SW103 SW_Push, SW104 SW_Push, SW105 SW_Push, SW106 SW_Push, SW107 SW_Push, SW108 SW_Push, SW109 SW_Push, SW110 SW_Push, SW111 SW_Push, SW112 SW_Push, SW113 SW_Push, SW114 SW_Push, SW115 SW_Push, SW116 SW_Push, SW117 SW_Push, SW118 SW_Push, SW119 SW_Push, SW120 SW_Push, SW121 SW_Push, SW122 SW_Push, SW123 SW_Push, SW124 SW_Push, SW125 SW_Push, SW2 RotaryEncoder_Switch, SW3 RotaryEncoder_Switch, SW71 SW_Push, SW72 SW_Push, SW73 SW_Push, SW74 SW_Push, SW75 SW_Push, SW76 SW_Push, SW77 SW_Push, SW78 SW_Push, SW79 SW_Push, SW80 SW_Push, SW81 SW_Push, SW82 SW_Push, SW83 SW_Push, SW84 SW_Push, SW85 SW_Push, SW86 SW_Push, SW87 SW_Push, SW88 SW_Push, SW89 SW_Push, SW90 SW_Push, SW91 SW_Push, SW92 SW_Push, SW93 SW_Push, SW94 SW_Push, SW95 SW_Push, SW96 SW_Push, SW97 SW_Push, SW98 SW_Push, SW99 SW_Push

Commit message: sync
Parts:
- A1: footprint Module:RaspberryPi_Pico_Common_SMD -> modded prints:RaspberryPi_Pico_Common_SMD noantenna
- D1, D10, D11, D12, D13, D14, D15, D16, D17, D18, D19, D2, D20, D21, D22, D23, D24, D25, D26, D27, D28, D29, D3, D30, D31, D32, D33, D34, D35, D36, D37, D38, D39, D4, D40, D41, D42, D43, D44, D45, D46, D47, D48, D49, D5, D50, D51, D52, D53, D54, D55, D56, D57, D58, D6, D7, D8, D9: footprint (none) -> Diode_SMD:D_0805_2012Metric_Pad1.15x1.40mm_HandSolder
- M1: footprint (none) -> Connector_PinHeader_1.00mm:PinHeader_1x02_P1.00mm_Vertical
- SW1, SW2, SW3: footprint (none) -> Rotary_Encoder:RotaryEncoder_Alps_EC11E-Switch_Vertical_H20mm
- SW100, SW101, SW102, SW103, SW104, SW105, SW106, SW107, SW108, SW109, SW110, SW111, SW112, SW113, SW114, SW115, SW116, SW117, SW118, SW119, SW123, SW124, SW125, SW71, SW72, SW73, SW74, SW75, SW76, SW79, SW80, SW81, SW82, SW83, SW84, SW85, SW86, SW87, SW88, SW89, SW90, SW91, SW92, SW93, SW94, SW95, SW96, SW97, SW98, SW99: footprint (none) -> ScottoKeebs_Hotswap:Hotswap_MX_1.00u
- SW120: footprint (none) -> ScottoKeebs_Hotswap:Hotswap_MX_2.00u
- SW121, SW122, SW77, SW78: footprint (none) -> ScottoKeebs_Hotswap:Hotswap_MX_1.50u
Connections:
- net c10: no longer SW3.S1
- net c12: now also SW3.S1
- no-connect marks 6 -> 7
